File: Placas/PCB Slave MMR1/Placa controladora carro mym.brd (EAGLE design)
At the start: 95 x 100 mm, 34 parts

Commit message: joystick funcionando
adicionado el control por joystick
Parts:
- D1, D2: value 1N4007 -> FR107
- moved 24V_IN 0.76 mm to (53.6, 94.2)
- renumbered REG_1 to REG_5V, REG_12 to REG_12V
Routing:
- net GND: track 357.6 -> 356.8 mm
Changed lines of the file:
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@@
 <?xml version="1.0" encoding="utf-8"?>
 <!DOCTYPE eagle SYSTEM "eagle.dtd">
-<eagle version="9.2.2">
+<eagle version="9.3.0">
 <drawing>
 <settings>
@@
 <attribute name="VALUE" x="80.438" y="63.373" size="1.27" layer="27"/>
 </element>
-<element name="24V_IN" library="pinhead" library_urn="urn:adsk.eagle:library:325" package="1X02" package3d_urn="urn:adsk.eagle:package:22435/2" value="" x="53.594" y="94.996" smashed="yes">
-<attribute name="NAME" x="50.9778" y="96.8248" size="1.27" layer="25" ratio="10"/>
-<attribute name="VALUE" x="51.054" y="91.821" size="1.27" layer="27"/>
-</element>
-<element name="D1" library="7DI Library" library_urn="urn:adsk.eagle:library:1229688" package="D-2.5" package3d_urn="urn:adsk.eagle:package:1237960/6" value="1N4007" x="26.416" y="74.422" smashed="yes">
-<attribute name="NAME" x="24.765" y="77.851" size="1.27" layer="25" ratio="10"/>
-<attribute name="VALUE" x="24.765" y="72.009" size="1.27" layer="27" ratio="10"/>
+<element name="24V_IN" library="pinhead" library_urn="urn:adsk.eagle:library:325" package="1X02" package3d_urn="urn:adsk.eagle:package:22435/2" value="" x="53.594" y="94.234" smashed="yes">
+<attribute name="NAME" x="50.9778" y="96.0628" size="1.27" layer="25" ratio="10"/>
+<attribute name="VALUE" x="51.054" y="91.059" size="1.27" layer="27"/>
+</element>
+<element name="D1" library="7DI Library" library_urn="urn:adsk.eagle:library:1229688" package="D-2.5" package3d_urn="urn:adsk.eagle:package:1237960/6" value="FR107" x="26.416" y="74.422" smashed="yes">
+<attribute name="NAME" x="29.337" y="70.485" size="1.27" layer="25" ratio="10"/>
+<attribute name="VALUE" x="29.337" y="73.279" size="1.27" layer="27" ratio="10"/>
 </element>
 <element name="5V1" library="pinhead" library_urn="urn:adsk.eagle:library:325" package="1X02" package3d_urn="urn:adsk.eagle:package:22435/2" value="" x="74.342" y="66.548" smashed="yes" rot="R180">
@@
 <attribute name="VALUE" x="23.5966" y="36.1696" size="0.9906" layer="27" ratio="10" rot="R270"/>
 </element>
-<element name="REG_12" library="arduino_nano" library_urn="urn:adsk.eagle:library:5132548" package="MOD_LM2596_FP" package3d_urn="urn:adsk.eagle:package:7198161/2" value="MOD_LM2596" x="24.384" y="87.122" smashed="yes">
-<attribute name="NAME" x="45.974" y="99.822" size="1.778" layer="26" rot="MR0"/>
-<attribute name="VALUE" x="12.954" y="73.152" size="1.778" layer="28" rot="MR0"/>
-</element>
-<element name="REG_1" library="arduino_nano" library_urn="urn:adsk.eagle:library:5132548" package="MOD_LM2596_FP" package3d_urn="urn:adsk.eagle:package:7198161/2" value="MOD_LM2596" x="24.384" y="61.722" smashed="yes">
-<attribute name="NAME" x="45.974" y="74.422" size="1.778" layer="26" rot="MR0"/>
-<attribute name="VALUE" x="11.938" y="45.72" size="1.778" layer="28" rot="MR0"/>
-</element>
-<element name="D2" library="7DI Library" library_urn="urn:adsk.eagle:library:1229688" package="D-2.5" package3d_urn="urn:adsk.eagle:package:1237960/6" value="1N4007" x="5.842" y="74.422" smashed="yes">
-<attribute name="NAME" x="4.191" y="75.565" size="1.27" layer="25" ratio="10"/>
-<attribute name="VALUE" x="4.191" y="72.009" size="1.27" layer="27" ratio="10"/>
+<element name="REG_12V" library="arduino_nano" library_urn="urn:adsk.eagle:library:5132548" package="MOD_LM2596_FP" package3d_urn="urn:adsk.eagle:package:7198161/2" value="MOD_LM2596" x="24.384" y="87.122" smashed="yes">
+<attribute name="NAME" x="41.656" y="92.202" size="1.778" layer="26" rot="MR0"/>
+<attribute name="VALUE" x="41.148" y="94.996" size="1.778" layer="28" rot="MR0"/>
+</element>
+<element name="REG_5V" library="arduino_nano" library_urn="urn:adsk.eagle:library:5132548" package="MOD_LM2596_FP" package3d_urn="urn:adsk.eagle:package:7198161/2" value="MOD_LM2596" x="24.384" y="61.722" smashed="yes">
+<attribute name="NAME" x="35.306" y="52.578" size="1.778" layer="26" rot="MR0"/>
+<attribute name="VALUE" x="35.306" y="55.626" size="1.778" layer="28" rot="MR0"/>
+</element>
+<element name="D2" library="7DI Library" library_urn="urn:adsk.eagle:library:1229688" package="D-2.5" package3d_urn="urn:adsk.eagle:package:1237960/6" value="FR107" x="5.842" y="74.422" smashed="yes">
+<attribute name="NAME" x="8.509" y="75.057" size="1.27" layer="25" ratio="10"/>
+<attribute name="VALUE" x="12.065" y="75.057" size="1.27" layer="27" ratio="10"/>
 </element>
 <element name="C7" library="7DI Library" library_urn="urn:adsk.eagle:library:1229688" package="CAP_CER_2,54-5X5" package3d_urn="urn:adsk.eagle:package:1281700/4" value="100nf" x="45.212" y="74.422" smashed="yes" rot="R180">
-<attribute name="NAME" x="47.498" y="72.898" size="1.27" layer="25" ratio="10" rot="R180"/>
-<attribute name="VALUE" x="47.498" y="77.216" size="1.27" layer="27" ratio="10" rot="R180"/>
+<attribute name="NAME" x="50.292" y="74.422" size="1.27" layer="25" ratio="10" rot="R270"/>
+<attribute name="VALUE" x="48.768" y="76.454" size="1.27" layer="27" ratio="10" rot="R270"/>
 </element>
 <element name="JP1" library="pinhead" library_urn="urn:adsk.eagle:library:325" package="1X06" package3d_urn="urn:adsk.eagle:package:22472/2" value="" x="70.866" y="94.234" smashed="yes">
@@
 <contactref element="R6" pad="1"/>
 <contactref element="R5" pad="1"/>
-<contactref element="REG_12" pad="IN-"/>
-<contactref element="REG_12" pad="OUT-"/>
+<contactref element="REG_12V" pad="IN-"/>
+<contactref element="REG_12V" pad="OUT-"/>
 <contactref element="12V1" pad="1"/>
 <contactref element="C5" pad="2"/>
 <contactref element="C3" pad="-"/>
 <contactref element="C6" pad="-"/>
-<contactref element="REG_1" pad="IN-"/>
-<contactref element="REG_1" pad="OUT-"/>
+<contactref element="REG_5V" pad="IN-"/>
+<contactref element="REG_5V" pad="OUT-"/>
 <contactref element="C7" pad="2"/>
 <contactref element="JP1" pad="2"/>
@@
 <wire x1="21.336" y1="34.036" x2="18.542" y2="34.036" width="0.4064" layer="16"/>
 <wire x1="24.13" y1="34.036" x2="21.336" y2="34.036" width="0.4064" layer="16"/>
-<wire x1="52.324" y1="94.996" x2="52.324" y2="89.916" width="0.4064" layer="16"/>
+<wire x1="52.324" y1="94.234" x2="52.324" y2="89.916" width="0.4064" layer="16"/>
 <wire x1="52.324" y1="89.916" x2="63.246" y2="89.916" width="0.4064" layer="16"/>
 <wire x1="63.246" y1="89.916" x2="65.786" y2="89.916" width="0.4064" layer="16"/>
@@
 <contactref element="C4" pad="1"/>
 <contactref element="D3" pad="A"/>
-<contactref element="REG_1" pad="OUT+"/>
+<contactref element="REG_5V" pad="OUT+"/>
 <contactref element="C7" pad="1"/>
 <contactref element="C" pad="3"/>
@@
 <contactref element="12V1" pad="2"/>
 <contactref element="C5" pad="1"/>
-<contactref element="REG_12" pad="OUT+"/>
+<contactref element="REG_12V" pad="OUT+"/>
 <wire x1="84.2734" y1="70.866" x2="84.2734" y2="66.5734" width="0.4064" layer="16"/>
 <wire x1="84.2734" y1="66.5734" x2="84.248" y2="66.548" width="0.4064" layer="16"/>
@@
 <contactref element="JP1" pad="1"/>
 <contactref element="CAM_PW" pad="4"/>
-<wire x1="54.864" y1="94.996" x2="59.69" y2="94.996" width="0.4064" layer="16"/>
-<wire x1="59.69" y1="94.996" x2="60.452" y2="94.234" width="0.4064" layer="16"/>
-<wire x1="60.452" y1="94.234" x2="64.516" y2="94.234" width="0.4064" layer="16"/>
+<wire x1="54.864" y1="94.234" x2="64.516" y2="94.234" width="0.4064" layer="16"/>
 <wire x1="27.686" y1="74.422" x2="27.686" y2="72.39" width="0.4064" layer="16"/>
 <wire x1="26.162" y1="70.866" x2="14.986" y2="70.866" width="0.4064" layer="16"/>
@@
 <wire x1="14.986" y1="44.45" x2="14.986" y2="70.866" width="0.4064" layer="16"/>
 <wire x1="9.8298" y1="39.2938" x2="14.986" y2="44.45" width="0.4064" layer="16"/>
-<wire x1="54.864" y1="94.996" x2="54.864" y2="96.774" width="0.4064" layer="16"/>
+<wire x1="54.864" y1="94.234" x2="54.864" y2="96.774" width="0.4064" layer="16"/>
 <wire x1="54.864" y1="96.774" x2="53.848" y2="97.79" width="0.4064" layer="16"/>
 <wire x1="53.848" y1="97.79" x2="49.784" y2="97.79" width="0.4064" layer="16"/>
@@
 <signal name="N$3">
 <contactref element="D1" pad="C"/>
-<contactref element="REG_12" pad="IN+"/>
+<contactref element="REG_12V" pad="IN+"/>
 <contactref element="C3" pad="+"/>
 <wire x1="25.146" y1="74.422" x2="18.542" y2="74.422" width="0.4064" layer="16"/>
@@
 </signal>
 <signal name="N$2">
-<contactref element="REG_1" pad="IN+"/>
+<contactref element="REG_5V" pad="IN+"/>
 <contactref element="C6" pad="+"/>
 <contactref element="D2" pad="C"/>
