File: Placas/PCB Slave MMR1/Placa controladora carro mym.sch (EAGLE design)
At the start: 34 parts

Commit message: joystick funcionando
adicionado el control por joystick
Parts:
- D1, D2: value 1N4007 -> FR107
- renumbered REG_1 to REG_5V, REG_12 to REG_12V
